File: BIPOv3.kicad_pcb (KiCad board)
At the start: 2 copper layers, 144.1 x 128 mm, 100 parts, among them J1 AudioJack2, J10 Conn_02x05_Odd_Even, J11 AudioJack2, J12 AudioJack2, J2 AudioJack2, J3 AudioJack2, J4 AudioJack2, J5 AudioJack2, J6 AudioJack2, J7 AudioJack2, J8 Conn_01x11_Pin, J9 Conn_01x11_Pin, Q1 BC857, Q2 BC857, SW1 SW_SPDT, U1 TL074, U18 LM13700, U2 TL074, U3 TL072

Commit message: Add files via upload
Parts:
- removed RV3, RV4: 500k, Potentiometer_THT:Potentiometer_ACP_CA9-H5_Horizontal
- added ?: , , F.Cu at (222.6, 97.8)
- added ?: , , F.Cu at (173.0, 98.0)
- added RV101: 500k, Potentiometer_THT:Potentiometer_Bourns_3266Y_Vertical, F.Cu at (207.2, 106.4)
- added RV102: 500k, Potentiometer_THT:Potentiometer_Bourns_3266Y_Vertical, F.Cu at (213.1, 106.4)
- moved ? 4.43 mm to (210.5, 127.2)
- moved C2 4.43 mm to (217.6, 101.9)
- moved J10 4.43 mm to (209.1, 134.4)
- moved R1 4.43 mm to (217.5, 94.7)
- moved R13 4.43 mm to (217.5, 97.1)
- moved R16 4.43 mm to (204.0, 120.7)
- moved R17 4.43 mm to (204.0, 118.3)
- moved R21 4.43 mm to (203.7, 98.8)
- moved R4 4.43 mm to (203.7, 93.8)
- moved R5 4.43 mm to (222.0, 109.5)
- moved R6 4.43 mm to (217.5, 99.5)
- moved J9 4.43 mm to (193.6, 96.3)
- moved R2 4.43 mm to (203.7, 101.1)
- moved R25 4.43 mm to (203.7, 96.2)
- moved R3 4.43 mm to (217.0, 92.3)
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Routing:
- net GND: track 27.0 -> 35.3 mm, vias 5 -> 6
- net Net-(R7-Pad2): track 8.57 -> 4.18 mm
- net Net-(U2D-+): track 28.6 -> 32.2 mm
- net Net-(U2A-+): track 32.1 -> 34.8 mm
- net Net-(R5-Pad2): track 10.4 -> 8.18 mm
- net Net-(R26-Pad1): track 96.4 -> 97.7 mm
- net Net-(D2-A): track 30.3 -> 31.3 mm
- net Net-(SW1-A): track 48.2 -> 49.0 mm
- net Net-(SW1-C): vias 1 -> 3
Other:
- board size 144.1 x 128 mm -> 139.6 x 128 mm
- board text added: "VCA1"
- board text added: "VCA2"
