File: BIPOv3.kicad_sch (KiCad schematic)
At the start: 78 parts, among them J1 AudioJack2, J10 Conn_02x05_Odd_Even, J11 AudioJack2, J12 AudioJack2, J2 AudioJack2, J3 AudioJack2, J4 AudioJack2, J5 AudioJack2, J6 AudioJack2, J7 AudioJack2, J8 Conn_01x11_Pin, J9 Conn_01x11_Pin, Q1 BC857, Q2 BC857, SW1 SW_SPDT, U1 TL074, U18 LM13700, U2 TL074, U3 TL072

Commit message: Add files via upload
Parts:
- removed RV3, RV4: 500k, Potentiometer_THT:Potentiometer_ACP_CA9-H5_Horizontal, symbol Device:R_Potentiometer
- added RV101, RV102: 500k, Potentiometer_THT:Potentiometer_Bourns_3266Y_Vertical, symbol Device:R_Potentiometer_Trim
- C1, C2, C3: value C -> 100n
Connections:
- net at R5.2: now also RV102.3
- net at R7.2: now also RV101.3
- net at R41.1, U18.5, U2.12 (+): now also RV101.1, RV101.2
- net at R38.1, U18.12, U2.3 (+): now also RV102.1, RV102.2
